Commit message: sim with nav stack now working. run roslaunch rover_launch rover_sim_launch.launch

File: src/rover_description/urdf/rover.xacro (robot description, xacro)
@@ -51,5 +51,5 @@
   <!-- BASE-FOOTPRINT -->
   <!-- base_footprint is a fictitious link(frame) that is on the ground right below base_link origin -->
-  <link name="base_footprint">
+<!--   <link name="base_footprint">
     <inertial>
       <mass value="0.0001" />
@@ -74,4 +74,5 @@
     <child link="base_link" />
   </joint>
+   -->
   <!-- BASE-LINK -->
   <!--Actual body/chassis of the robot-->
@@ -168,5 +169,5 @@
   <!-- SENSORS -->
   <!-- hokuyo -->
-  <link name="hokuyo_link">
+  <link name="base_laser">
     <visual>
       <origin xyz="0 0 0" rpy="0 0 0" />
@@ -180,7 +181,7 @@
     <origin xyz="${base_radius - hokuyo_size/2} 0 ${base_height+hokuyo_size/4}" rpy="0 0 0" />
     <parent link="base_link"/>
-    <child link="hokuyo_link" />
-  </joint>
-  <gazebo reference="hokuyo_link">
+    <child link="base_laser" />
+  </joint>
+  <gazebo reference="base_laser">
     <material>Gazebo/Blue</material>
     <turnGravityOff>false</turnGravityOff>
@@ -188,5 +189,5 @@
       <pose>${hokuyo_size/2} 0 0 0 0 0</pose>
       <visualize>true</visualize>
-      <update_rate>40</update_rate>
+      <update_rate>20</update_rate>
       <ray>
         <scan>
@@ -206,5 +207,5 @@
       <plugin name="gazebo_ros_head_hokuyo_controller" filename="libgazebo_ros_laser.so">
         <topicName>/scan</topicName>
-        <frameName>hokuyo_link</frameName>
+        <frameName>base_laser</frameName>
       </plugin>
     </sensor>
@@ -215,8 +216,8 @@
       <rosDebugLevel>Debug</rosDebugLevel>
       <publishWheelTF>false</publishWheelTF>
-      <legacyMode>false</legacyMode>
-      <robotNamespace>/</robotNamespace>
+<!--       <legacyMode>false</legacyMode>
+ -->      <robotNamespace>/</robotNamespace>
       <publishTf>1</publishTf>
-      <publishWheelJointState>false</publishWheelJointState>
+      <publishWheelJointState>true</publishWheelJointState>
       <alwaysOn>true</alwaysOn>
       <updateRate>100.0</updateRate>
@@ -229,4 +230,5 @@
       <wheelAcceleration>1.8</wheelAcceleration>
       <commandTopic>cmd_vel</commandTopic>
+      <odometrySource>world-</odometrySource>
       <odometryFrame>odom</odometryFrame>
       <odometryTopic>odom</odometryTopic>

Commit message: added downward facing laser to model. actual rover model coming SOON

File: src/rover_description/urdf/rover.xacro (robot description, xacro)
@@ -179,5 +179,5 @@
   </link>
   <joint name="hokuyo_joint" type="fixed">
-    <origin xyz="${base_radius - hokuyo_size/2} 0 ${base_height+hokuyo_size/4}" rpy="0 0 0" />
+    <origin xyz="${-1*base_radius - hokuyo_size/2} 0 ${base_height+hokuyo_size/4}" rpy="0 0 ${M_PI}" />
     <parent link="base_link"/>
     <child link="base_laser" />
@@ -211,4 +211,46 @@
     </sensor>
   </gazebo>
+  <link name="front_laser">
+    <visual>
+      <origin xyz="0 0 0" rpy="0 0 0" />
+      <geometry>
+        <mesh filename="package://rover_description/meshes/hokuyo.dae"/>
+      </geometry>
+      <material name="Blue" />
+    </visual>
+  </link>
+  <joint name="front_hokuyo_joint" type="fixed">
+    <origin xyz="${base_radius - hokuyo_size/2} 0 ${.1+base_height+hokuyo_size/4}" rpy="0 .3 0" />
+    <parent link="base_link"/>
+    <child link="front_laser" />
+  </joint>
+  <gazebo reference="front_laser">
+    <material>Gazebo/Blue</material>
+    <turnGravityOff>false</turnGravityOff>
+    <sensor type="ray" name="front_hokuyo_sensor">
+      <pose>${hokuyo_size/2} 0 0 0 0 0</pose>
+      <visualize>true</visualize>
+      <update_rate>20</update_rate>
+      <ray>
+        <scan>
+          <horizontal>
+            <samples>720</samples>
+            <resolution>1</resolution>
+            <min_angle>-1.570796</min_angle>
+            <max_angle>1.570796</max_angle>
+          </horizontal>
+        </scan>
+        <range>
+          <min>0.10</min>
+          <max>10.0</max>
+          <resolution>0.001</resolution>
+        </range>
+      </ray>
+      <plugin name="gazebo_ros_head_hokuyo_controller" filename="libgazebo_ros_laser.so">
+        <topicName>/front_scan</topicName>
+        <frameName>front_laser</frameName>
+      </plugin>
+    </sensor>
+  </gazebo>
   <!-- Differential drive controller  -->
   <gazebo>

Commit message: edits

File: src/rover_description/urdf/rover.xacro (robot description, xacro)
@@ -169,5 +169,5 @@
   <!-- SENSORS -->
   <!-- hokuyo -->
-  <link name="base_laser">
+  <link name="back_laser">
     <visual>
       <origin xyz="0 0 0" rpy="0 0 0" />
@@ -179,9 +179,9 @@
   </link>
   <joint name="hokuyo_joint" type="fixed">
-    <origin xyz="${-1*base_radius - hokuyo_size/2} 0 ${base_height+hokuyo_size/4}" rpy="0 0 ${M_PI}" />
-    <parent link="base_link"/>
-    <child link="base_laser" />
-  </joint>
-  <gazebo reference="base_laser">
+    <origin xyz="${-1*base_radius + hokuyo_size/2} 0 ${base_height+hokuyo_size/4}" rpy="0 0 ${M_PI}" />
+    <parent link="base_link"/>
+    <child link="back_laser" />
+  </joint>
+  <gazebo reference="back_laser">
     <material>Gazebo/Blue</material>
     <turnGravityOff>false</turnGravityOff>
@@ -206,6 +206,6 @@
       </ray>
       <plugin name="gazebo_ros_head_hokuyo_controller" filename="libgazebo_ros_laser.so">
-        <topicName>/scan</topicName>
-        <frameName>base_laser</frameName>
+        <topicName>/back_scan</topicName>
+        <frameName>back_laser</frameName>
       </plugin>
     </sensor>

Commit message: amcl workin\'

File: src/rover_description/urdf/rover.xacro (robot description, xacro)
@@ -221,5 +221,5 @@
   </link>
   <joint name="front_hokuyo_joint" type="fixed">
-    <origin xyz="${base_radius - hokuyo_size/2} 0 ${.1+base_height+hokuyo_size/4}" rpy="0 .3 0" />
+    <origin xyz="${base_radius - hokuyo_size/2} 0 ${.1+base_height+hokuyo_size/4}" rpy="0 .2 0" />
     <parent link="base_link"/>
     <child link="front_laser" />
@@ -253,4 +253,38 @@
     </sensor>
   </gazebo>
+  <link name="imu_link">
+    <inertial>
+      <mass value="0.1"/>
+      <origin xyz="0 0 0" />
+      <cylinder_inertia  m="0.1" r="0.03" h="0.03" />
+    </inertial>
+    <visual name="visual">
+      <origin xyz="0 0 0" rpy="0 0 0" />
+      <geometry>
+        <box size="0.03 0.03 0.03"/>
+      </geometry>
+    </visual>
+    <collision name="collision">
+    <origin xyz="0 0 0" rpy="0 0 0" />
+      <geometry>
+        <box size="0.03 0.03 0.03"/>
+      </geometry>
+    </collision>
+  </link>
+  <joint name="imu_joint" type="fixed">
+    <origin xyz="0 0 .0" rpy="0 0 0" />
+    <parent link="base_link"/>
+    <child link="imu_link" />
+  </joint>
+  <gazebo reference="imu_link">
+      <plugin name="imu_plugin" filename="libgazebo_ros_imu.so">
+          <alwaysOn>true</alwaysOn>
+          <bodyName>imu_link</bodyName>
+          <topicName>/imu_data</topicName>
+          <serviceName>/simu_service</serviceName>
+          <gaussianNoise>0.0</gaussianNoise>
+          <updateRate>10.0</updateRate>
+      </plugin>
+  </gazebo>
   <!-- Differential drive controller  -->
   <gazebo>

Commit message: Fixed imu sim

File: src/rover_description/urdf/rover.xacro (robot description, xacro)
@@ -253,37 +253,41 @@
     </sensor>
   </gazebo>
+  <joint name="imu_joint" type="fixed">
+    <axis xyz="1 0 0"/> <!-- 0 1 0 -->
+    <origin xyz="0 0 0"/>
+    <parent link="base_link"/>
+    <child link="imu_link"/>
+  </joint>
   <link name="imu_link">
     <inertial>
-      <mass value="0.1"/>
-      <origin xyz="0 0 0" />
-      <cylinder_inertia  m="0.1" r="0.03" h="0.03" />
-    </inertial>
-    <visual name="visual">
-      <origin xyz="0 0 0" rpy="0 0 0" />
+      <mass value="0.001"/>
+      <origin rpy="0 0 0" xyz="0 0 0"/>
+      <inertia ixx="0.0001" ixy="0" ixz="0" iyy="0.000001" iyz="0" izz="0.0001"/>
+    </inertial>
+    <visual>
+      <origin rpy="0 0 0" xyz="0 0 0"/>
       <geometry>
         <box size="0.03 0.03 0.03"/>
       </geometry>
     </visual>
-    <collision name="collision">
-    <origin xyz="0 0 0" rpy="0 0 0" />
-      <geometry>
-        <box size="0.03 0.03 0.03"/>
+    <collision>
+      <origin rpy="0 0 0" xyz="0 0 0"/>
+      <geometry>
+        <box size=".03 .03 .03"/>
       </geometry>
     </collision>
   </link>
-  <joint name="imu_joint" type="fixed">
-    <origin xyz="0 0 .0" rpy="0 0 0" />
-    <parent link="base_link"/>
-    <child link="imu_link" />
-  </joint>
-  <gazebo reference="imu_link">
-      <plugin name="imu_plugin" filename="libgazebo_ros_imu.so">
-          <alwaysOn>true</alwaysOn>
-          <bodyName>imu_link</bodyName>
-          <topicName>/imu_data</topicName>
-          <serviceName>/simu_service</serviceName>
-          <gaussianNoise>0.0</gaussianNoise>
-          <updateRate>10.0</updateRate>
-      </plugin>
+  <gazebo>
+    <plugin name="imu_controller" filename="libgazebo_ros_imu.so">
+      <alwaysOn>true</alwaysOn>
+      <updateRate>50.0</updateRate>
+      <bodyName>imu_link</bodyName>
+      <topicName>imu_data</topicName>
+      <frameName>imu_link</frameName>
+      <serviceName>imu_service</serviceName>
+      <gaussianNoise>2.89e-08</gaussianNoise>
+      <xyzOffsets>0 0 0</xyzOffsets>
+      <rpyOffsets>0 0 0</rpyOffsets>
+    </plugin>
   </gazebo>
   <!-- Differential drive controller  -->

Commit message: adding config files for using robot localization

File: src/rover_description/urdf/rover.xacro (robot description, xacro)
@@ -29,10 +29,10 @@
   <!-- caster wheel mass -->
   <xacro:property name="caster_f_height" value="0.04" />
-  <xacro:property name="caster_f_radius" value="0.025" />
+  <xacro:property name="caster_f_radius" value="0.027" />
   <xacro:property name="caster_f_mass" value="0.5" /> <!-- in kg-->
   <!-- caster wheel radius and height -->
   <!-- caster wheel mass -->
   <xacro:property name="caster_b_height" value="0.04" />
-  <xacro:property name="caster_b_radius" value="0.025" />
+  <xacro:property name="caster_b_radius" value="0.027" />
   <xacro:property name="caster_b_mass" value="0.5" /> <!-- in kg-->
   <!-- Wheels -->
@@ -179,5 +179,5 @@
   </link>
   <joint name="hokuyo_joint" type="fixed">
-    <origin xyz="${-1*base_radius + hokuyo_size/2} 0 ${base_height+hokuyo_size/4}" rpy="0 0 ${M_PI}" />
+    <origin xyz="${-1*base_radius + hokuyo_size/2} 0 ${.1+base_height+hokuyo_size/4}" rpy="0 0 ${M_PI}" />
     <parent link="base_link"/>
     <child link="back_laser" />
@@ -312,5 +312,5 @@
       <odometrySource>world-</odometrySource>
       <odometryFrame>odom</odometryFrame>
-      <odometryTopic>gazebo/odom</odometryTopic>
+      <odometryTopic>/gazebo/odom</odometryTopic>
       <robotBaseFrame>base_footprint</robotBaseFrame>
     </plugin>

Commit message: adding configs still messed...

File: src/rover_description/urdf/rover.xacro (robot description, xacro)
@@ -51,5 +51,5 @@
   <!-- BASE-FOOTPRINT -->
   <!-- base_footprint is a fictitious link(frame) that is on the ground right below base_link origin -->
-<!--   <link name="base_footprint">
+  <link name="base_footprint">
     <inertial>
       <mass value="0.0001" />
@@ -71,8 +71,7 @@
   <joint name="base_footprint_joint" type="fixed">
     <origin xyz="0 0 ${wheel_radius - base_z_origin_to_wheel_origin}" rpy="0 0 0" />
-    <parent link="base_footprint"/>
-    <child link="base_link" />
-  </joint>
-   -->
+    <parent link="base_link"/>
+    <child link="base_footprint" />
+  </joint>
   <!-- BASE-LINK -->
   <!--Actual body/chassis of the robot-->
@@ -310,8 +309,8 @@
       <wheelAcceleration>1.8</wheelAcceleration>
       <commandTopic>cmd_vel</commandTopic>
-      <odometrySource>world-</odometrySource>
-      <odometryFrame>odom</odometryFrame>
+      <odometrySource>world</odometrySource>
+      <odometryFrame>/gazebo/odom</odometryFrame>
       <odometryTopic>/gazebo/odom</odometryTopic>
-      <robotBaseFrame>base_footprint</robotBaseFrame>
+      <robotBaseFrame>/gazebo/base_link</robotBaseFrame>
     </plugin>
   </gazebo>
